Commit message: Updates to allow single robot and twin robots to be spawned in Gazebo. -Still a few kinks to work out with planning scene

File: ur5e_2f85/ur5e_2f85_description/urdf/robotiq_wrist_camera.urdf.xacro (robot description, xacro)
@@ -35,5 +35,6 @@
       <parent link="${prefix}robotiq_wrist_camera_base_link"/>
       <child link="${prefix}robotiq_wrist_camera_frame"/>
-      <origin rpy="${-pi/2} ${-pi/2} ${-pi/2}" xyz="0.05 0.0 0.01"/>
+      <!-- <origin rpy="${-pi/2} ${-pi/2} ${-pi/2}" xyz="0.05 0.0 0.01"/> -->
+      <origin rpy="0 ${-pi/2 + 0.3} 0" xyz="0.05 0.0 0.01"/> <!-- Pitch by an extra 0.3 radians to account for wrist camera angle -->
     </joint>
     <link name="${prefix}robotiq_wrist_camera_frame">

File: ur5e_2f85/ur5e_2f85_description/urdf/ur5e_2f85_joint_limited_robot.urdf.xacro (robot description, xacro)
@@ -1,4 +1,4 @@
 <?xml version="1.0"?>
-<robot xmlns:xacro="http://wiki.ros.org/xacro"
+<robot xmlns:xacro="http://www.ros.org/wiki/xacro"
        name="ur5e_2f85" >
   <!-- Simulated flag -->
@@ -7,20 +7,4 @@
   <xacro:property name="use_grasp_fix" value="false"/>
   <xacro:arg name="prefix" default=""/>
-  <!--
-  <xacro:arg name="base_x" default="1.0"/>
-  <xacro:arg name="base_y" default="1.0"/>
-  <xacro:arg name="base_z" default="1.0"/>
-  <xacro:arg name="base_R" default="1.0"/>
-  <xacro:arg name="base_P" default="1.0"/>
-  <xacro:arg name="base_Y" default="1.0"/>
-  -->
-  <!--
-  <xacro:property name="base_x" value="$(arg base_x)" />
-  <xacro:property name="base_y" value="$(arg base_y)" />
-  <xacro:property name="base_z" value="$(arg base_z)" />
-  <xacro:property name="base_R" value="$(arg base_R)" />
-  <xacro:property name="base_P" value="$(arg base_P)" />
-  <xacro:property name="base_Y" value="$(arg base_Y)" />
-  -->
   <!-- The transmission interface to use for UR5e -->
   <xacro:arg name="transmission_hw_interface" default="hardware_interface/PositionJointInterface"/>
@@ -48,5 +32,5 @@
   <xacro:include filename="$(find robotiq_2f_85_gripper_visualization)/urdf/robotiq_arg2f_85_model_macro.xacro" />
   <xacro:robotiq_arg2f_85 prefix="$(arg prefix)"/>
-  <joint name="robotiq_wrist_camera_ee_joint" type="fixed">
+  <joint name="robotiq_wrist_camera_arg2f_joint" type="fixed">
     <parent link="robotiq_wrist_camera_base_link" />
     <child link = "robotiq_arg2f_base_link"/>

Commit message: Added wrist camera urdf

File: ur5e_2f85/ur5e_2f85_description/urdf/robotiq_wrist_camera.urdf.xacro (robot description, xacro)
@@ -9,5 +9,5 @@
     <link name="${prefix}robotiq_wrist_camera_base_link">
       <inertial>
-        <origin rpy="0 0 0" xyz="0 0 ${-17 / 1000}"/>
+        <origin rpy="0 0 0" xyz="0 0 0"/>
         <mass value="0.300"/>
         <inertia ixx="${262 / 1000000}" ixy="0" ixz="${1 / 1000000}" iyx="0" iyy="${265 / 1000000}" iyz="${1 / 1000000}" izx="${-1 / 1000000}" izy="${1 / 1000000}" izz="${219 / 1000000}"/>
@@ -17,5 +17,5 @@
         <geometry>
           <!--<mesh filename="package://uncalibrated_grasping/models/other_models/robotiq_wrist_camera/meshes/robotiq_wrist_camera.STL"/>-->
-          <cylinder length="0.02" radius="0.05"/>
+          <cylinder length="0.02" radius="0.04"/>
           <mesh filename="package://ur5e_2f85_description/meshes/robotiq_wrist_camera.STL"/>
         </geometry>
@@ -28,5 +28,5 @@
         <geometry>
           <!--<mesh filename="package://uncalibrated_grasping/models/other_models/robotiq_wrist_camera/meshes/robotiq_wrist_camera.STL"/>-->
-          <cylinder length="0.02" radius="0.05"/>
+          <cylinder length="0.02" radius="0.04"/>
         </geometry>
       </collision>
@@ -34,9 +34,9 @@
     <joint name="${prefix}robotiq_wrist_camera_base_camera_frame_joint" type="fixed">
       <parent link="${prefix}robotiq_wrist_camera_base_link"/>
-      <child link="${prefix}robotiq_wrist_camera_frame"/>
+      <child link="${prefix}robotiq_wrist_camera_link"/>
       <!-- <origin rpy="${-pi/2} ${-pi/2} ${-pi/2}" xyz="0.05 0.0 0.01"/> -->
-      <origin rpy="0 ${-pi/2 + 0.3} 0" xyz="0.05 0.0 0.01"/> <!-- Pitch by an extra 0.3 radians to account for wrist camera angle -->
+      <origin rpy="${pi/2} ${-pi/2} ${-pi/2}" xyz="0.00 0.0 0.015"/> <!-- Pitch by an extra 0.3 radians to account for wrist camera angle -->
     </joint>
-    <link name="${prefix}robotiq_wrist_camera_frame">
+    <link name="${prefix}robotiq_wrist_camera_link">
       <inertial>
         <origin rpy="0 0 0" xyz="0 0 0"/>
@@ -46,5 +46,5 @@
       <visual>
         <origin rpy="0 0 0" xyz="0 0 0"/>
-        <geometry>`
+        <geometry>
           <box size="0.005 0.005 0.005"/>
         </geometry>
@@ -60,5 +60,21 @@
       </collision>
     </link>
-    <gazebo reference="${prefix}robotiq_wrist_camera_frame">
+    <link name="robotiq_wrist_camera_link_optical">
+    </link>
+    <joint name="camera_optical_joint" type="fixed">
+      <!-- these values have to be these values otherwise the gazebo camera
+          image won't be aligned properly with the frame it is supposedly
+          originating from -->
+      <origin xyz="0 0 0" rpy="${-pi/2} 0 ${-pi/2}"/>
+      <parent link="robotiq_wrist_camera_link"/>
+      <child link="robotiq_wrist_camera_link_optical"/>
+    </joint>
+    <link name="robotiq_wrist_camera_frame"/>
+    <joint name="tool0_robotiq_wrist_camera_frame" type="fixed">
+      <origin xyz="0 0 0" rpy="${pi} 0 0"/>
+      <parent link="tool0"/>
+      <child link="robotiq_wrist_camera_frame"/>
+    </joint>
+    <gazebo reference="robotiq_wrist_camera_link">
       <sensor name="openni_camera_camera" type="depth">
         <always_on>1</always_on>
@@ -80,6 +96,6 @@
           <alwaysOn>true</alwaysOn>
           <updateRate>30.0</updateRate>
-          <cameraName>robotiq_wrist_camera</cameraName>
-          <frameName>${prefix}robotiq_wrist_camera_frame</frameName>
+          <cameraName>wrist_camera</cameraName>
+          <frameName>robotiq_wrist_camera_link_optical</frameName>
           <imageTopicName>image</imageTopicName>
           <depthImageTopicName>depth/image_raw</depthImageTopicName>
